Commit message: Update wsg_50.urdf.xacro

File: wsg50_gripper/urdf/wsg_50.urdf.xacro (robot description, xacro)
@@ -65,5 +65,5 @@
   <!-- LEFT FINGER -->
   <joint name="${name}_guide_joint_finger_left" type="fixed">
-     <origin xyz="${finger_tip} 0 ${finger_length}" rpy="0 0 0" />
+     <origin xyz="0 0 0" rpy="0 0 0" />
      <parent link="${name}_gripper_left"/>
      <child link="${name}_finger_left" />
@@ -128,5 +128,5 @@
   <!-- RIGHT FINGER -->
   <joint name="${name}_guide_joint_finger_right" type="fixed">
-     <origin xyz="${finger_tip} 0 ${finger_length}" rpy="0 0 0" />
+     <origin xyz="0 0 0" rpy="0 0 0" />
      <parent link="${name}_gripper_right"/>
      <child link="${name}_finger_right" />
